File: epi_ESP32 (2023_01_16 13_30_41 UTC).kicad_pcb (KiCad board)
At the start: 4 copper layers, 12.7 x 36 mm, 61 parts, among them J1 Conn_01x08, J2 USB_C_Receptacle_USB2.0, J3 Conn_01x08, J5 Conn_01x06, Q1 Q_PMOS_GDS, Q2 Q_NMOS_GDS, Q3 Q_NMOS_GDS, Q4 Q_NMOS_GDS, Q5 Q_NMOS_GDS, Q6 Q_NMOS_GDS, SW1 SW_MEC_5G, SW2 SW_MEC_5G, U1 ESP32-C3, U2 MIC5219-5.0YM5, U4 MIC5219-3.3YM5, Y1 Crystal

Commit message: init
Parts:
- added J4: Conn_01x02, Connector_PinHeader_2.54mm:PinHeader_1x02_P2.54mm_Vertical, F.Cu at (118.5, 48.9)
